Commit message: check nav2 param

File: metu_description/urdf/rover_gazebo_imu.xacro (robot description, xacro)
@@ -4,5 +4,5 @@
     <parent link="chassis" />
     <child link="imu_link" />
-    <origin xyz="0 0 0.20" rpy="0 0 0" />
+    <origin xyz="0 0 0.20" rpy="0 0 0" /><!-- 0 0 ${-pi}-->
   </joint>
   <link name="imu_link">
@@ -26,5 +26,5 @@
           <remapping>~/out:=imu</remapping>
         </ros>
-        <initial_orientation_as_reference>true</initial_orientation_as_reference>
+        <initial_orientation_as_reference>false</initial_orientation_as_reference>
         <frame_name>imu_link</frame_name>
       </plugin>

File: metu_description/urdf/rover_gps.xacro (robot description, xacro)
@@ -24,5 +24,5 @@
             <ros>
                 <!-- <namespace>/br</namespace> -->
-                <remapping>gps_controller/out:=gps</remapping>
+                <remapping>gps_controller/out:=gps/fix</remapping>
             </ros>
             <frame_name>gps_link</frame_name>
