Commit message: gps nav2 works

File: metu_description/urdf/rover_depth.xacro (robot description, xacro)
@@ -4,5 +4,5 @@
         <parent link="chassis" />
         <child link="camera_link" />
-        <origin xyz="0.3 0 0.1" rpy="0 0 0" /><!-- 0 0.38 -0.2      0 0 ${pi/2}-->
+        <origin xyz="0.3 0 0.1" rpy="0 0 0" /><!-- 0 0.38 -0.2      0 0 ${pi/2}--> <!-- 0.3 0 0.1-->
     </joint>
     <link name="camera_link">
@@ -20,5 +20,5 @@
         <parent link="camera_link" />
         <child link="camera_link_optical" />
-        <origin xyz="0 0 0" rpy="${-pi/2} 0 ${-pi/2}" /><!-- ${pi/2} ${pi} ${pi/2}--><!-- ${-pi/2} 0 ${-pi/2}-->
+        <origin xyz="0 0 0" rpy="${-pi/2} 0 ${-pi/2}" /><!-- ${pi/2} ${pi} ${pi/2}--><!-- ${-pi/2} 0 ${-pi/2}--><!-- 0 0 0-->
     </joint>
     <link name="camera_link_optical">

File: metu_description/urdf/rover_gazebo_imu.xacro (robot description, xacro)
@@ -4,5 +4,5 @@
     <parent link="chassis" />
     <child link="imu_link" />
-    <origin xyz="0 0 0.20" rpy="0 0 0" /><!-- 0 0 ${-pi}-->
+    <origin xyz="0 0 0.20" rpy="0 0 0" /><!-- 0 0 ${-pi}--> <!-- 0 0 0-->
   </joint>
   <link name="imu_link">
